File: HDK/Lite/1Job.kicad_sch (KiCad schematic)
At the start: 9 parts, among them U101 STM32G030K6Tx, U102 AMS1117-3.3

Commit message: updated 1 Job, WIP
Parts:
- removed R101, R102: 5.1k, Resistor_SMD:R_0603_1608Metric, symbol Device:R
Connections:
- net CAN_CS1: now also U101.27 (PB3); no longer U101.11 (PA4)
- net DO_SSR: now reaches U101.16 (PB1)
- net PC6: now reaches U101.20 (PC6)
- net PA15: now reaches U101.26 (PA15)
- net PB4: now reaches U101.28 (PB4)
- net PB5: now reaches U101.29 (PB5)
- net ANA_0 renamed PA0
- net SDCARD_CS renamed PA8
- net SPI1_MISO renamed PA6
- net SPI1_MOSI renamed PA7
- net SPI1_SCK renamed PA5
- net SPI2_MISO renamed PB2
- net SPI2_MOSI renamed PA10
- net SPI2_SCK renamed PB8
- net SWCLK renamed PA14
- net SWDIO renamed PA13
- net UART1_RX renamed PB7
- net UART1_TX renamed PB6
- net UART2_RX renamed PA3
- net UART2_TX renamed PA2
- new net PA4: U101.11 (PA4)
- no-connect marks 2 -> 9
