File: HDK/Lite/CanBus.kicad_sch (KiCad schematic)
At the start: 10 parts, among them J201 TERM, U201 SN65HVD230, U202 MCP2518FD, Y201 40MHz

Commit message: updated 1 Job
Parts:
- removed C106 (x2): 100n, Capacitor_SMD:C_0603_1608Metric, symbol Device:C
- added C106 (x2): 100n, Capacitor_SMD:C_0603_1608Metric, symbol Device:C
Connections:
- net +3V3: now also C106.1, C106.1
- net GND: now also C106.2, C106.2

Commit message: updated 1-Job, v1rA
Parts:
- removed Y201: 40MHz, Crystal:Crystal_SMD_3225-4Pin_3.2x2.5mm, symbol Device:Crystal_GND23_Small
- added Y201: 40MHz, Crystal:Crystal_SMD_3225-4Pin_3.2x2.5mm, symbol Device:Crystal_GND24_Small
- C106: LCSC (none) -> C57112
- C203, C204: value 10p -> 20p; LCSC (none) -> C1648
- J201: footprint Connector_PinHeader_2.54mm:PinHeader_1x02_P2.54mm_Vertical -> Connector_PinHeader_2.54mm:PinHeader_1x02_P2.54mm_Horizontal
- R201: LCSC (none) -> C25804
- R202: LCSC (none) -> C22787
- U201: LCSC (none) -> C12084
- U202: LCSC (none) -> C626758
Connections:
- net CAN_+: now also J201.2 (Pin_2); no longer J201.1 (Pin_1)
- net GND: now also Y201.2, Y201.4
- net OSC_IN: now also Y201.3
- net OSC_OUT: now also Y201.1
- net at R202.1: now also J201.1 (Pin_1); no longer J201.2 (Pin_2)
Changed lines of the file:
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@@
+    (stroke (width 0) (type default))
+  )
+  (wire (pts (xy 215.9 96.52) (xy 203.2 96.52))
     (stroke (width 0) (type default))
   )
@@
     (stroke (width 0) (type default))
   )
+  (wire (pts (xy 203.2 99.06) (xy 227.33 99.06))
+    (stroke (width 0) (type default))
+  )
   (wire (pts (xy 182.88 85.09) (xy 171.45 85.09))
     (stroke (width 0) (type default))
@@
     (stroke (width 0) (type default))
   )
-  (wire (pts (xy 223.52 99.06) (xy 227.33 99.06))
-    (stroke (width 0) (type default))
-  )
   (wire (pts (xy 85.09 88.9) (xy 85.09 87.63))
     (stroke (width 0) (type default))
@@
     (stroke (width 0) (type default))
   )
-  (wire (pts (xy 203.2 96.52) (xy 227.33 96.52))
-    (stroke (width 0) (type default))
-  )
   (wire (pts (xy 110.49 97.79) (xy 121.92 97.79))
     (stroke (width 0) (type default))
@@
     (stroke (width 0) (type default))
   )
-  (wire (pts (xy 215.9 99.06) (xy 203.2 99.06))
+  (wire (pts (xy 223.52 96.52) (xy 227.33 96.52))
     (stroke (width 0) (type default))
   )
@@
     (effects (font (size 1.27 1.27)) (justify right bottom))
   )
+  (label "CAN_-" (at 203.2 96.52 0) (fields_autoplaced)
+    (effects (font (size 1.27 1.27)) (justify left bottom))
+  )
   (label "SPI_CANCS" (at 110.49 87.63 0) (fields_autoplaced)
     (effects (font (size 1.27 1.27)) (justify left bottom))
@@
     (effects (font (size 1.27 1.27)) (justify right bottom))
   )
+  (label "CAN_+" (at 203.2 99.06 0) (fields_autoplaced)
+    (effects (font (size 1.27 1.27)) (justify left bottom))
+  )
   (label "CAN_RX" (at 171.45 85.09 0) (fields_autoplaced)
     (effects (font (size 1.27 1.27)) (justify left bottom))
@@
   (label "CAN_TX" (at 163.83 85.09 180) (fields_autoplaced)
     (effects (font (size 1.27 1.27)) (justify right bottom))
-  )
-  (label "CAN_+" (at 203.2 96.52 0) (fields_autoplaced)
-    (effects (font (size 1.27 1.27)) (justify left bottom))
-  )
-  (label "CAN_-" (at 203.2 99.06 0) (fields_autoplaced)
-    (effects (font (size 1.27 1.27)) (justify left bottom))
   )
   (hierarchical_label "CAN_+" (shape input) (at 214.63 85.09 0) (fields_autoplaced)
@@
       (effects (font (size 1.27 1.27)) hide)
     )
-    (property "LCSC" "" (at 193.04 85.09 0)
+    (property "LCSC" "C12084" (at 193.04 85.09 0)
       (effects (font (size 1.27 1.27)) hide)
     )
@@
     )
   )
-  (symbol (lib_id "Device:R") (at 219.71 99.06 270) (mirror x) (unit 1)
-    (in_bom yes) (on_board yes) (dnp no)
-    (property "Reference" "R202" (at 214.63 97.79 90)
-      (effects (font (size 1.27 1.27)))
-    )
-    (property "Value" "120" (at 224.79 100.33 90)
-      (effects (font (size 1.27 1.27)))
-    )
-    (property "Footprint" "Resistor_SMD:R_0603_1608Metric" (at 219.71 100.838 90)
-      (effects (font (size 1.27 1.27)) hide)
-    )
-    (property "Datasheet" "~" (at 219.71 99.06 0)
-      (effects (font (size 1.27 1.27)) hide)
-    )
-    (property "LCSC" "" (at 219.71 99.06 0)
-      (effects (font (size 1.27 1.27)) hide)
-    )
-    (pin "1")
-    (pin "2")
-    (instances
-      (project "1Job"
-        (path "/250934e5-fe91-4d13-9aa6-67dcfb888854/ea28d679-3f64-46ea-8bdc-1fa483262ea5"
-          (reference "R202") (unit 1)
-        )
-      )
-    )
-  )
   (symbol (lib_id "Device:C_Small") (at 77.47 91.44 0) (mirror y) (unit 1)
     (in_bom yes) (on_board yes) (dnp no) (fields_autoplaced)
@@
       (effects (font (size 1.27 1.27)) (justify left))
     )
-    (property "Value" "10p" (at 74.93 92.7163 0)
+    (property "Value" "20p" (at 74.93 92.7163 0)
       (effects (font (size 1.27 1.27)) (justify left))
     )
@@
       (effects (font (size 1.27 1.27)) hide)
     )
-    (property "LCSC" "" (at 77.47 91.44 0)
+    (property "LCSC" "C1648" (at 77.47 91.44 0)
       (effects (font (size 1.27 1.27)) hide)
     )
@@
       (effects (font (size 1.27 1.27)) (justify left))
     )
-    (property "Value" "10p" (at 87.63 92.7163 0)
+    (property "Value" "20p" (at 87.63 92.7163 0)
       (effects (font (size 1.27 1.27)) (justify left))
     )
@@
       (effects (font (size 1.27 1.27)) hide)
     )
-    (property "LCSC" "" (at 85.09 91.44 0)
+    (property "LCSC" "C1648" (at 85.09 91.44 0)
       (effects (font (size 1.27 1.27)) hide)
     )
@@
       (effects (font (size 1.27 1.27)) hide)
     )
-    (property "LCSC" "" (at 127 68.58 0)
+    (property "LCSC" "C57112" (at 127 68.58 0)
       (effects (font (size 1.27 1.27)) hide)
     )
@@
       (effects (font (size 1.27 1.27)) (justify left))
     )
-    (property "Footprint" "Connector_PinHeader_2.54mm:PinHeader_1x02_P2.54mm_Vertical" (at 232.41 96.52 0)
+    (property "Footprint" "Connector_PinHeader_2.54mm:PinHeader_1x02_P2.54mm_Horizontal" (at 232.41 96.52 0)
       (effects (font (size 1.27 1.27)) hide)
     )
@@
       (effects (font (size 1.27 1.27)) hide)
     )
-    (property "LCSC" "" (at 179.07 95.25 0)
+    (property "LCSC" "C25804" (at 179.07 95.25 0)
       (effects (font (size 1.27 1.27)) hide)
     )
@@
       (effects (font (size 1.27 1.27)) hide)
     )
-    (property "LCSC" "" (at 137.16 90.17 0)
+    (property "LCSC" "C626758" (at 137.16 90.17 0)
       (effects (font (size 1.27 1.27)) hide)
     )
@@
       (effects (font (size 1.27 1.27)) hide)
     )
-    (property "LCSC" "" (at 182.88 68.58 0)
+    (property "LCSC" "C57112" (at 182.88 68.58 0)
       (effects (font (size 1.27 1.27)) hide)
     )
@@
         (path "/250934e5-fe91-4d13-9aa6-67dcfb888854/ea28d679-3f64-46ea-8bdc-1fa483262ea5"
           (reference "#PWR0206") (unit 1)
+        )
+      )
+    )
+  )
+  (symbol (lib_id "Device:R") (at 219.71 96.52 270) (unit 1)
+    (in_bom yes) (on_board yes) (dnp no)
+    (property "Reference" "R202" (at 214.63 97.79 90)
+      (effects (font (size 1.27 1.27)))
+    )
+    (property "Value" "120" (at 224.79 95.25 90)
+      (effects (font (size 1.27 1.27)))
+    )
+    (property "Footprint" "Resistor_SMD:R_0603_1608Metric" (at 219.71 94.742 90)
+      (effects (font (size 1.27 1.27)) hide)
+    )
+    (property "Datasheet" "~" (at 219.71 96.52 0)
+      (effects (font (size 1.27 1.27)) hide)
+    )
+    (property "LCSC" "C22787" (at 219.71 96.52 0)
+      (effects (font (size 1.27 1.27)) hide)
+    )
+    (pin "1")
+    (pin "2")
+    (instances
+      (project "1Job"
+        (path "/250934e5-fe91-4d13-9aa6-67dcfb888854/ea28d679-3f64-46ea-8bdc-1fa483262ea5"
+          (reference "R202") (unit 1)
         )
       )
@@
     )
   )
-  (symbol (lib_id "Device:Crystal_GND23_Small") (at 81.28 87.63 0) (unit 1)
+  (symbol (lib_id "Device:Crystal_GND24_Small") (at 81.28 87.63 0) (unit 1)
     (in_bom yes) (on_board yes) (dnp no)
-    (property "Reference" "Y201" (at 86.36 81.28 0)
-      (effects (font (size 1.27 1.27)))
-    )
-    (property "Value" "40MHz" (at 86.36 83.82 0)
+    (property "Reference" "Y201" (at 86.36 80.01 0)
+      (effects (font (size 1.27 1.27)))
+    )
+    (property "Value" "40MHz" (at 86.36 82.55 0)
       (effects (font (size 1.27 1.27)))
     )
@@
       (effects (font (size 1.27 1.27)) hide)
     )
-    (property "LCSC" "" (at 81.28 87.63 0)
-      (effects (font (size 1.27 1.27)) hide)
-    )
-    (pin "1")
-    (pin "2")
+    (property "LCSC" "C9010" (at 81.28 87.63 0)
+      (effects (font (size 1.27 1.27)) hide)
+    )
     (pin "3")
     (pin "4")
-    (instances
-      (project "1Job"
+    (pin "2")
+    (pin "1")
+    (instances
+      (project "1Job"

Commit message: updated 1job
Other:
- company: (none) -> Scott CJX
- title: (none) -> 1 Job Lite
Changed lines of the file:
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@@
 (kicad_sch (version 20230121) (generator eeschema)
   (paper "A4")
+  (title_block
+    (title "1 Job Lite")
+    (date "2023-11-13")
+    (rev "A")
+    (company "Scott CJX")
+  )
   (junction (at 85.09 87.63) (diameter 0) (color 0 0 0 0)
   )
