File: HDK/Lite/SDCard.kicad_sch (KiCad schematic)
At the start: 1 part, among them J301 Micro_SD_Card_Det1

Commit message: updated 1 Job
Parts:
- J301: value Micro_SD_Card_Det1 -> GT-TF003-H0185-02; footprint (none) -> Connector_Card:microSD_HC_Molex_104031-0811; LCSC (none) -> C5155564
Changed lines of the file:
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@@
   (symbol (lib_id "power:GND") (at 95.25 96.52 270) (unit 1)
     (in_bom yes) (on_board yes) (dnp no) (fields_autoplaced)
-    (property "Reference" "#PWR0301" (at 88.9 96.52 0)
+    (property "Reference" "#PWR0302" (at 88.9 96.52 0)
       (effects (font (size 1.27 1.27)) hide)
     )
@@
     (pin "1")
     (instances
-      (project "ControllerLite"
+      (project "1Job"
         (path "/250934e5-fe91-4d13-9aa6-67dcfb888854/614c74f4-d8d1-4546-8dcf-6b150dd58bfd"
-          (reference "#PWR0301") (unit 1)
+          (reference "#PWR0302") (unit 1)
         )
       )
@@
       (effects (font (size 1.27 1.27)))
     )
-    (property "Value" "Micro_SD_Card_Det1" (at 135.255 74.93 0)
+    (property "Value" "GT-TF003-H0185-02" (at 135.255 74.93 0)
       (effects (font (size 1.27 1.27)))
     )
-    (property "Footprint" "" (at 186.69 76.2 0)
+    (property "Footprint" "Connector_Card:microSD_HC_Molex_104031-0811" (at 186.69 76.2 0)
       (effects (font (size 1.27 1.27)) hide)
     )
     (property "Datasheet" "https://datasheet.lcsc.com/lcsc/2110151630_XKB-Connectivity-XKTF-015-N_C381082.pdf" (at 134.62 91.44 0)
+      (effects (font (size 1.27 1.27)) hide)
+    )
+    (property "LCSC" "C5155564" (at 134.62 93.98 0)
       (effects (font (size 1.27 1.27)) hide)
     )
@@
     (pin "9")
     (instances
-      (project "ControllerLite"
+      (project "1Job"
         (path "/250934e5-fe91-4d13-9aa6-67dcfb888854/614c74f4-d8d1-4546-8dcf-6b150dd58bfd"
           (reference "J301") (unit 1)
@@
   (symbol (lib_id "power:+3V3") (at 95.25 91.44 90) (unit 1)
     (in_bom yes) (on_board yes) (dnp no)
-    (property "Reference" "#PWR0302" (at 99.06 91.44 0)
+    (property "Reference" "#PWR0301" (at 99.06 91.44 0)
       (effects (font (size 1.27 1.27)) hide)
     )
@@
     (pin "1")
     (instances
-      (project "ControllerLite"
+      (project "1Job"
         (path "/250934e5-fe91-4d13-9aa6-67dcfb888854/614c74f4-d8d1-4546-8dcf-6b150dd58bfd"
-          (reference "#PWR0302") (unit 1)
+          (reference "#PWR0301") (unit 1)
         )
       )
@@
     (pin "1")
     (instances
-      (project "ControllerLite"
+      (project "1Job"
         (path "/250934e5-fe91-4d13-9aa6-67dcfb888854/614c74f4-d8d1-4546-8dcf-6b150dd58bfd"
           (reference "#PWR0303") (unit 1)

Commit message: updated 1-Job, v1rA
Parts:
- removed J301: GT-TF003-H0185-02, Connector_Card:microSD_HC_Molex_104031-0811, symbol Connector:Micro_SD_Card_Det1
- added J302: DM3CS-SF, footprints:HRS_DM3CS-SF, symbol DM3CS-SF:DM3CS-SF
Connections:
- net +3V3: now also J302.4 (VDD)
- net GND: now also J302.6 (VSS), J302.S1 (GND), J302.S2 (GND), J302.S3 (GND), J302.S5 (GND)
- net SD_DET: now also J302.9 (CD_SW)
- net SPI_CLK: now also J302.5 (CLK)
- net SPI_MISO: now also J302.7 (DAT0)
- net SPI_MOSI: now also J302.3 (CMD)
- net SPI_SDCS: now also J302.2 (CD/DAT3)

Commit message: updated 1job
Other:
- company: (none) -> Scott CJX
- title: (none) -> 1 Job Lite
Changed lines of the file:
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@@
 (kicad_sch (version 20230121) (generator eeschema)
   (paper "A4")
+  (title_block
+    (title "1 Job Lite")
+    (date "2023-11-13")
+    (rev "A")
+    (company "Scott CJX")
+  )
   (no_connect (at 115.57 142.24))
   (no_connect (at 115.57 139.7))

Commit message: updated BOM, wip
Parts:
- J302: AVAILABILITY Good -> (none); Availability In Stock -> (none); Check_prices https://www.snapeda.com/parts/DM3CS-SF/Hirose+Electric+Co+L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 -> (none); DESCRIPTION CONN MICRO SD CARD HINGED TYPE -> (none); LCSC (none) -> C202111; MANUFACTURER Hirose -> (none); MF Hirose Electric Co Ltd -> (none); MP DM3CS-SF -> (none); PACKAGE None -> (none); PARTREV n/a -> (none); PRICE 1.14 USD -> (none); Package None -> (none); Price None -> (none); Purchase-URL https://www.snapeda.com/api/url_track_click_mouser/?unipart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 -> (none); STANDARED manufacturer recommendation -> (none); SnapEDA_Link https://www.snapeda.com/parts/DM3CS-SF/Hirose+Electric+Co+L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 -> (none)
Changed lines of the file:
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@@
       (effects (font (size 1.27 1.27)) hide)
     )
-    (property "MF" "Hirose Electric Co Ltd" (at 128.27 137.16 0)
-      (effects (font (size 1.27 1.27)) (justify bottom) hide)
+    (property "LCSC" "C202111" (at 128.27 137.16 0)
+      (effects (font (size 1.27 1.27)) hide)
     )
-    (property "DESCRIPTION" "CONN MICRO SD CARD HINGED TYPE" (at 128.27 137.16 0)
-      (effects (font (size 1.27 1.27)) (justify bottom) hide)
-    )
-    (property "PACKAGE" "None" (at 128.27 137.16 0)
-      (effects (font (size 1.27 1.27)) (justify bottom) hide)
-    )
-    (property "PRICE" "1.14 USD" (at 128.27 137.16 0)
-      (effects (font (size 1.27 1.27)) (justify bottom) hide)
-    )
-    (property "Package" "None" (at 128.27 137.16 0)
-      (effects (font (size 1.27 1.27)) (justify bottom) hide)
-    )
-    (property "Check_prices" "https://www.snapeda.com/parts/DM3CS-SF/Hirose+Electric+Co+Ltd/view-part/?ref=eda" (at 128.27 137.16 0)
-      (effects (font (size 1.27 1.27)) (justify bottom) hide)
-    )
-    (property "Availability" "In Stock" (at 128.27 137.16 0)
-      (effects (font (size 1.27 1.27)) (justify bottom) hide)
-    )
-    (property "Price" "None" (at 128.27 137.16 0)
-      (effects (font (size 1.27 1.27)) (justify bottom) hide)
-    )
-    (property "PARTREV" "n/a" (at 128.27 137.16 0)
-      (effects (font (size 1.27 1.27)) (justify bottom) hide)
-    )
-    (property "SnapEDA_Link" "https://www.snapeda.com/parts/DM3CS-SF/Hirose+Electric+Co+Ltd/view-part/?ref=snap" (at 128.27 137.16 0)
-      (effects (font (size 1.27 1.27)) (justify bottom) hide)
-    )
-    (property "MP" "DM3CS-SF" (at 128.27 137.16 0)
-      (effects (font (size 1.27 1.27)) (justify bottom) hide)
-    )
-    (property "Purchase-URL" "https://www.snapeda.com/api/url_track_click_mouser/?unipart_id=12308516&manufacturer=Hirose Electric Co Ltd&part_name=DM3CS-SF&search_term=None" (at 128.27 137.16 0)
-      (effects (font (size 1.27 1.27)) (justify bottom) hide)
-    )
-    (property "Description" "\n10 (8 + 2) Position Card Connector Secure Digital - microSD™ Surface Mount, Right Angle Gold\n" (at 128.27 137.16 0)
-      (effects (font (size 1.27 1.27)) (justify bottom) hide)
-    )
-    (property "STANDARED" "manufacturer recommendation" (at 128.27 137.16 0)
-      (effects (font (size 1.27 1.27)) (justify bottom) hide)
-    )
-    (property "AVAILABILITY" "Good" (at 128.27 137.16 0)
-      (effects (font (size 1.27 1.27)) (justify bottom) hide)
-    )
-    (property "MANUFACTURER" "Hirose" (at 128.27 137.16 0)
-      (effects (font (size 1.27 1.27)) (justify bottom) hide)
-    )
-    (pin "9")
-    (pin "5")
+    (pin "1")
+    (pin "2")
     (pin "3")
     (pin "4")
+    (pin "5")
     (pin "6")
-    (pin "S3")
     (pin "7")
+    (pin "8")
+    (pin "9")
     (pin "S1")
     (pin "S2")
-    (pin "1")
+    (pin "S3")
     (pin "S5")
-    (pin "8")
-    (pin "2")
     (instances
       (project "1Job"
